Commit message: Make PLZ fixed

File: x3plus_description/urdf/yahboomcar_X3plusX.urdf.xacro (robot description, xacro)
@@ -3,4 +3,7 @@
     xmlns:gz="http://gazebosim.org/schema">
     <!-- define the list of relevant args -->
+    <xacro:arg name="fixedPLZJoints" default="true" />
+    <!-- set the internal properties based on the arguments -->
+    <xacro:property name="fixedPLZJoints" value="$(arg fixedPLZJoints)" />
     <!-- <xacro:if value="${namespace == 'None'}">
         <xacro:property name="ns" value="" />
@@ -198,7 +201,13 @@
         </inertial>
     </xacro:common_link>
-    <xacro:revolute_joint name="arm_joint1" parent="base_link" child="arm_link1"
+    <xacro:if value="${fixedPLZJoints}">
+        <xacro:fixed_joint name="arm_joint1" parent="base_link" child="arm_link1"
+        xyz="0.09825 0 0.102" rpy="0 0 0" />
+    </xacro:if>
+    <xacro:unless value="${fixedPLZJoints}">
+        <xacro:revolute_joint name="arm_joint1" parent="base_link" child="arm_link1"
         xyz="0.09825 0 0.102" rpy="0 0 0" axisZ="-1"
         lower="-${pi/2}" upper="${pi/2}" />
+    </xacro:unless>
     <xacro:common_link name="arm_link2b" material="Green" path="X3plus">
         <inertial>
@@ -214,6 +223,12 @@
         </inertial>
     </xacro:common_link>
-    <xacro:revolute_joint name="arm_joint2" parent="arm_link1" child="arm_link2b" xyz="0 0 0.0405"
+    <xacro:if value="${fixedPLZJoints}">
+        <xacro:fixed_joint name="arm_joint2" parent="arm_link1" child="arm_link2b" xyz="0 0 0.0405"
+        rpy="-${pi/2} 0 0"   />
+    </xacro:if>
+    <xacro:unless value="${fixedPLZJoints}">
+        <xacro:revolute_joint name="arm_joint2" parent="arm_link1" child="arm_link2b" xyz="0 0 0.0405"
         rpy="-${pi/2} 0 0" axisZ="-1" lower="-${pi/2}" upper="${pi/2}" />
+    </xacro:unless>
     <xacro:fixed_joint name="camera_joint" parent="arm_link2b" child="camera_link" xyz="0 -0.07 0"
         rpy="${pi/2} 0 0" />
@@ -416,5 +431,6 @@
         child="back_right_wheel"
         xyz="-0.115 -0.103 -0.038" rpy="${pi/2} 0 ${pi}" axis="0 0 1" />
-    <xacro:wheel_continuous_joint name="back_left_joint" parent="base_link" child="back_left_wheel"
+    <xacro:wheel_continuous_joint name="back_left_joint" parent="base_link"
+        child="back_left_wheel"
         xyz="-0.115  0.103 -0.038" rpy="${pi/2} 0 0" axis="0 0 1" />
    <gazebo>
@@ -429,17 +445,17 @@
                 <wheelbase>0.16</wheelbase>
                 <!-- Wheel radius -->
-                <wheel_radius>-0.042</wheel_radius>
+                <wheel_radius>0.042</wheel_radius>
                 <!-- <min_acceleration>-5</min_acceleration>
                 <max_acceleration>5</max_acceleration> -->
-                <max_velocity>3.0</max_velocity>
-                <min_velocity>-3.0</min_velocity>
+                <!-- <max_velocity>3.0</max_velocity>
+                <min_velocity>-3.0</min_velocity> -->
                 <!-- <min_jerk>3</min_jerk>
                 <max_jerk>-3</max_jerk> -->
-                <odom_publish_frequency>10</odom_publish_frequency>
+                <!-- <odom_publish_frequency>10</odom_publish_frequency>
                 <odom_topic>/odometry</odom_topic>
                 <publish_odom_tf>false</publish_odom_tf>
                 <publish_wheel_tf>true</publish_wheel_tf>
                 <topic>/cmd_vel</topic>
-                <tf_topic>/pose</tf_topic>
+                <tf_topic>/pose</tf_topic> -->
             </plugin>
         </gazebo>
@@ -516,5 +532,5 @@
             <visualize>true</visualize>
             <topic>imu</topic>
-            <gz_frame_id>base_link</gz_frame_id>
+            <frame_id >base_link</frame_id >
             <imu>
                 <angular_velocity>
@@ -578,5 +594,5 @@
         <topic>lidar</topic>
         <update_rate>10</update_rate>
-        <gz_frame_id>laser_link</gz_frame_id>
+        <frame_id >laser_link</frame_id >
         <ray>
                 <scan>
@@ -611,5 +627,5 @@
             <topic>/color/image_raw</topic>
             <visualize>true</visualize>
-            <gz_frame_id>camera_link</gz_frame_id>
+            <frame_id >camera_link</frame_id >
             <horizontal_fov>${60.0/180.0*pi}</horizontal_fov>
             <image>
@@ -627,6 +643,6 @@
             <topic>/depth/image_raw</topic>
             <visualize>true</visualize>
-            <!-- <gz_frame_id>camera_link</gz_frame_id> -->
-            <gz_frame_id>camera_link_optical</gz_frame_id>
+            <!-- <frame_id >camera_link</frame_id > -->
+            <frame_id >camera_link_optical</frame_id >
             <camera>
                 <horizontal_fov>${60.0/180.0*pi}</horizontal_fov>
@@ -651,6 +667,6 @@
             <topic>/color/opt/image_raw</topic>
             <visualize>true</visualize>
-            <!-- <gz_frame_id>camera_link</gz_frame_id> -->
-            <gz_frame_id>camera_link_optical</gz_frame_id>
+            <!-- <frame_id >camera_link</frame_id > -->
+            <frame_id >camera_link_optical</frame_id >
             <horizontal_fov>${60.0/180.0*pi}</horizontal_fov>
             <image>
@@ -668,6 +684,6 @@
             <topic>/depth/opt/image_raw</topic>
             <visualize>true</visualize>
-            <!-- <gz_frame_id>camera_link</gz_frame_id> -->
-            <gz_frame_id>camera_link_optical</gz_frame_id>
+            <!-- <frame_id >camera_link</frame_id > -->
+            <frame_id >camera_link_optical</frame_id >
             <camera>
                 <horizontal_fov>${60.0/180.0*pi}</horizontal_fov>

Commit message: fixing transforms of the wheeels

File: x3plus_description/urdf/yahboomcar_X3plusX.urdf.xacro (robot description, xacro)
@@ -118,5 +118,5 @@
                 <pose>0 0 0 0 0 0</pose>
                 <geometry>
-                    <sphere radius="0.032391999999999997" />
+                    <sphere radius="0.04" />
                 </geometry>
             </collision>
@@ -427,5 +427,5 @@
     <xacro:wheel_continuous_joint name="front_left_joint" parent="base_link"
         child="front_left_wheel"
-        xyz="0.105   0.103 -0.038" rpy="${pi/2} 0 0" axis="0 0 1" />
+        xyz="0.105   0.103 -0.038" rpy="-${pi/2} 0 0" axis="0 0 1" />
     <xacro:wheel_continuous_joint name="back_right_joint" parent="base_link"
         child="back_right_wheel"
@@ -433,5 +433,5 @@
     <xacro:wheel_continuous_joint name="back_left_joint" parent="base_link"
         child="back_left_wheel"
-        xyz="-0.115  0.103 -0.038" rpy="${pi/2} 0 0" axis="0 0 1" />
+        xyz="-0.115  0.103 -0.038" rpy="-${pi/2} 0 0" axis="0 0 1" />
    <gazebo>
             <plugin name='gz::sim::systems::MecanumDrive' filename='gz-sim-mecanum-drive-system'>
@@ -441,21 +441,22 @@
                 <back_right_joint>back_right_joint</back_right_joint>
                 <!-- Lateral distance between left and right wheels -->
-                <wheel_separation>0.169</wheel_separation>
+                 <!-- end 2 end is 245.6 mm ; width of the wheel is 37.4 ==> 0.2082 -->
+                <wheel_separation>0.2082</wheel_separation>
                 <!-- Longitudinal distance between front and back wheels -->
-                <wheelbase>0.16</wheelbase>
+                <wheelbase>0.22</wheelbase>
                 <!-- Wheel radius -->
-                <wheel_radius>0.042</wheel_radius>
-                <!-- <min_acceleration>-5</min_acceleration>
-                <max_acceleration>5</max_acceleration> -->
+                <wheel_radius>0.040</wheel_radius>
+                <min_acceleration>-5</min_acceleration>
+                <max_acceleration>5</max_acceleration>
                 <!-- <max_velocity>3.0</max_velocity>
                 <min_velocity>-3.0</min_velocity> -->
                 <!-- <min_jerk>3</min_jerk>
                 <max_jerk>-3</max_jerk> -->
-                <!-- <odom_publish_frequency>10</odom_publish_frequency>
+                <odom_publish_frequency>10</odom_publish_frequency>
                 <odom_topic>/odometry</odom_topic>
                 <publish_odom_tf>false</publish_odom_tf>
                 <publish_wheel_tf>true</publish_wheel_tf>
                 <topic>/cmd_vel</topic>
-                <tf_topic>/pose</tf_topic> -->
+                <tf_topic>/pose</tf_topic>
             </plugin>
         </gazebo>

Commit message: Update Lidar meshes

File: x3plus_description/urdf/yahboomcar_X3plusX.urdf.xacro (robot description, xacro)
@@ -173,4 +173,5 @@
         <inertial>
             <origin xyz="-0.0176558922685589 0.000671805271544437 0.0219302095894866" rpy="0 0 0" />
+            <!-- <origin xyz="-0.0176558922685589 0.000671805271544437 0.0219302095894866" rpy="0 0 0" /> -->
             <mass value="0.0483909504209895" />
             <inertia ixx="1.58456966399128E-05" ixy="-4.23913983850005E-07"
@@ -180,5 +181,6 @@
     </xacro:common_link>
     <xacro:fixed_joint name="laser_joint" parent="base_link" child="laser_link"
-        xyz="0.10478 0 0.0471" rpy="0 0 0" />
+        xyz="0.10478 0 0" rpy="0 0 0" />
+        <!-- xyz="0.10478 0 0.0471" rpy="0 0 0" /> -->
     <xacro:common_link name="camera_link" material="White" path="sensor">
         <inertial>
@@ -621,6 +623,6 @@
                     </scan>
                     <range>
-                        <min>0.08</min>
-                        <max>10.0</max>
+                        <min>0.05</min>
+                        <max>12.0</max>
                         <resolution>0.01</resolution>
                     </range>

Commit message: Add IMU Links

File: x3plus_description/urdf/yahboomcar_X3plusX.urdf.xacro (robot description, xacro)
@@ -56,5 +56,4 @@
         <origin xyz="0.0 0.0 0.076" rpy="0 0 0" />
     </joint>
-    <!-- <link name="imu_link"/> -->
     <!-- common link-->
     <xacro:macro name="common_link" params="name material path *origin">
@@ -168,6 +167,9 @@
     <fixed_joint name="base_joint" parent="base_footprint" child="base_link" xyz="0.0 0.0 0.076" rpy="0
     0 0"/> -->
-    <!-- <fixed_joint name="base_imu" parent="base_link" child="imu_link" xyz="0.001 0.017 0.0322"
-    rpy="0 3.1415 1.5707"/> -->
+    <link name="imu_link"/>
+    <xacro:fixed_joint name="base_imu" parent="base_link" child="imu_link" xyz="0 0 0"
+        rpy="0 0 0"/>
+    <!-- <xacro:fixed_joint name="base_imu" parent="base_link" child="imu_link" xyz="0.001 0.017 0.0322"
+        rpy="0 3.1415 1.5707"/>  -->
     <xacro:common_link name="laser_link" material="White" path="sensor">
         <inertial>
@@ -535,6 +537,8 @@
             <visualize>true</visualize>
             <topic>imu</topic>
-            <!-- <frame_id >base_link</frame_id > -->
-            <gz_frame_id>base_link</gz_frame_id >
+            <gz_frame_id>base_link</gz_frame_id>
+            <!-- <gz_frame_id>imu_link</gz_frame_id> -->
+            <!-- Set whether to output orientation. Not all imu's generate orientation values as they use filters to produce orientation estimates. -->
+            <!-- <orientation_enabled>false</orientation_enabled> -->
             <imu>
                 <angular_velocity>
@@ -593,4 +597,31 @@
         </sensor>
     </gazebo>
+     <!-- <sensor name="magnetometer" type="magnetometer">
+          <always_on>1</always_on>
+          <update_rate>100</update_rate>
+          <visualize>true</visualize>
+          <topic>magnetometer</topic>
+          <enable_metrics>true</enable_metrics>
+          <magnetometer>
+            <x>
+              <noise type="gaussian">
+                <mean>0.0</mean>
+                <stddev>0.1</stddev>
+              </noise>
+            </x>
+            <y>
+              <noise type="gaussian">
+                <mean>0.0</mean>
+                <stddev>0.1</stddev>
+              </noise>
+            </y>
+            <z>
+              <noise type="gaussian">
+                <mean>0.0</mean>
+                <stddev>0.1</stddev>
+              </noise>
+            </z>
+          </magnetometer>
+        </sensor> -->
     <gazebo reference="laser_link">
         <sensor name='gpu_lidar' type='gpu_lidar'>

Commit message: Adding laser support

File: x3plus_description/urdf/yahboomcar_X3plusX.urdf.xacro (robot description, xacro)
@@ -172,5 +172,6 @@
     <xacro:fixed_joint name="base_imu" parent="base_link" child="imu_link" xyz="0.001 0.017 0.0322"
         rpy="0 3.1415 1.5707"/>
-    <xacro:common_link name="laser_link" material="White" path="sensor">
+   <link name="laser_link"/>
+    <xacro:common_link name="sllidar_link" material="White" path="sensor">
         <inertial>
             <origin xyz="-0.0176558922685589 0.000671805271544437 0.0219302095894866" rpy="0 0 0" />
@@ -182,6 +183,8 @@
         </inertial>
     </xacro:common_link>
-    <xacro:fixed_joint name="laser_joint" parent="base_link" child="laser_link"
+    <xacro:fixed_joint name="sllidar_joint" parent="base_link" child="sllidar_link"
         xyz="0.10478 0 0" rpy="0 0 0" />
+        <xacro:fixed_joint name="laser_joint" parent="base_link" child="laser_link"
+        xyz="0.10478 0 0.035" rpy="0 0 0" />
         <!-- xyz="0.10478 0 0.0471" rpy="0 0 0" /> -->
     <xacro:common_link name="camera_link" material="White" path="sensor">
@@ -644,6 +647,10 @@
                             <samples>640</samples>
                             <resolution>1</resolution>
+                            <min_angle>-3.14159</min_angle>
+                            <max_angle>3.14159</max_angle>
+                            <!--
                             <min_angle>-1.396263</min_angle>
                             <max_angle>1.396263</max_angle>
+                            -->
                         </horizontal>
                         <vertical>
