Commit message: Adjust URDF name

File: x3plus_description/urdf/yahboomcar_X3plus.urdf.xacro (robot description, xacro)
@@ -1,6 +1,11 @@
 <?xml version="1.0" encoding="utf-8"?>
-<robot name="yahboomcar_X3plus" xmlns:xacro="http://wiki.ros.org/xacro" xmlns:gz="http://gazebosim.org/schema">
-  <!-- define the list of relevant args -->
-  <!-- <xacro:if value="${namespace == 'None'}">
+<robot name="yahboomcar_X3plus" xmlns:xacro="http://wiki.ros.org/xacro"
+    xmlns:gz="http://gazebosim.org/schema">
+    <!-- define the list of relevant args -->
+    <xacro:arg name="fixedPLZJoints" default="true" />
+    <xacro:arg name="fixedPLZJoints" default="true"  />
+    <!-- set the internal properties based on the arguments -->
+    <xacro:property name="fixedPLZJoints" value="$(arg fixedPLZJoints)" />
+    <!-- <xacro:if value="${namespace == 'None'}">
         <xacro:property name="ns" value="" />
       </xacro:if>
@@ -9,28 +14,29 @@
       </xacro:unless> -->
     <material name="Green">
-        <color rgba="0 0.7 0 1"/>
+        <color rgba="0 0.7 0 1" />
     </material>
     <material name="White">
-        <color rgba="0.7 0.7 0.7 1"/>
+        <color rgba="0.7 0.7 0.7 1" />
     </material>
-    <xacro:property name="ns" value="$(arg ns)"/>
+    <xacro:property name="ns" value="$(arg ns)" />
     <xacro:property name="wheel_radius" value="0.05" />
-    <link name="base_footprint"/>
+    <link name="base_footprint" />
     <link name="base_link">
         <inertial>
-            <origin xyz="-0.0304416859098744 4.23384368655101E-05 0.0448234503408059" rpy="0 0 0"/>
-            <mass value="1.0754239466482"/>
-            <inertia
-                    ixx="0.0208831789264125"
-                    ixy="2.4618093127858E-06"
-                    ixz="0.00616019290028669"
-                    iyy="0.0265621377486244"
-                    iyz="-1.10079499865282E-06"
-                    izz="0.0129535610833954"/>
+            <origin xyz="-0.0304416859098744 4.23384368655101E-05 0.0448234503408059" rpy="0 0 0" />
+            <mass value="1.0754239466482" />
+            <inertia
+                ixx="0.0208831789264125"
+                ixy="2.4618093127858E-06"
+                ixz="0.00616019290028669"
+                iyy="0.0265621377486244"
+                iyz="-1.10079499865282E-06"
+                izz="0.0129535610833954" />
         </inertial>
         <visual>
             <origin xyz="0 0 0" rpy="0 0 0" />
             <geometry>
-                    <mesh filename="package://x3plus_description/meshes/X3plus/visual/base-link-core.STL"/>
+                <mesh
+                    filename="package://x3plus_description/meshes/X3plus/visual/base-link-small.STL" />
             </geometry>
             <material name="">
@@ -41,5 +47,6 @@
             <origin xyz="0 0 0" rpy="0 0 0" />
             <geometry>
-                    <mesh filename="package://x3plus_description/meshes/X3plus/collision/base-link-core.STL"/>
+                <mesh
+                    filename="package://x3plus_description/meshes/X3plus/collision/base-link-small.STL" />
             </geometry>
         </collision>
@@ -50,5 +57,4 @@
         <origin xyz="0.0 0.0 0.076" rpy="0 0 0" />
     </joint>
-    <!-- <link name="imu_link"/> -->
     <!-- common link-->
     <xacro:macro name="common_link" params="name material path *origin">
@@ -56,16 +62,17 @@
             <visual>
                 <geometry>
-                    <mesh filename="package://x3plus_description/meshes/${path}/visual/${name}.STL"/>
+                    <mesh filename="package://x3plus_description/meshes/${path}/visual/${name}.STL" />
                 </geometry>
-                <origin xyz="0 0 0" rpy="0 0 0"/>
-                <material name="${material}"/>
+                <origin xyz="0 0 0" rpy="0 0 0" />
+                <material name="${material}" />
             </visual>
             <collision>
                 <geometry>
-                    <mesh filename="package://x3plus_description/meshes/${path}/collision/${name}.STL"/>
+                    <mesh
+                        filename="package://x3plus_description/meshes/${path}/collision/${name}.STL" />
                 </geometry>
-                <origin xyz="0 0 0" rpy="0 0 0"/>
+                <origin xyz="0 0 0" rpy="0 0 0" />
             </collision>
-            <xacro:insert_block name="origin"/>
+            <xacro:insert_block name="origin" />
         </link>
     </xacro:macro>
@@ -73,9 +80,9 @@
     <xacro:macro name="revolute_joint" params="name parent child xyz rpy axisZ lower upper">
         <joint name="${name}" type="revolute">
-            <parent link="${parent}"/>
-            <child link="${child}"/>
-            <origin xyz="${xyz}" rpy="${rpy}"/>
-            <axis xyz="0 0 ${axisZ}"/>
-            <limit lower="${lower}" upper="${upper}" effort="100" velocity="1"/>
+            <parent link="${parent}" />
+            <child link="${child}" />
+            <origin xyz="${xyz}" rpy="${rpy}" />
+            <axis xyz="0 0 ${axisZ}" />
+            <limit lower="${lower}" upper="${upper}" effort="100" velocity="1" />
         </joint>
     </xacro:macro>
@@ -83,9 +90,9 @@
     <xacro:macro name="continuous_joint" params="name parent child xyz rpy mimic">
         <joint name="${name}" type="continuous">
-            <parent link="${parent}"/>
-            <child link="${child}"/>
-            <origin xyz="${xyz}" rpy="${rpy}"/>
-            <axis xyz="0 0 1"/>
-            <mimic joint="grip_joint" multiplier="${mimic}"/>
+            <parent link="${parent}" />
+            <child link="${child}" />
+            <origin xyz="${xyz}" rpy="${rpy}" />
+            <axis xyz="0 0 1" />
+            <mimic joint="grip_joint" multiplier="${mimic}" />
         </joint>
     </xacro:macro>
@@ -93,10 +100,10 @@
     <xacro:macro name="fixed_joint" params="name parent child xyz rpy">
         <joint name="${name}" type="fixed">
-            <parent link="${parent}"/>
-            <child link="${child}"/>
-            <origin xyz="${xyz}" rpy="${rpy}"/>
+            <parent link="${parent}" />
+            <child link="${child}" />
+            <origin xyz="${xyz}" rpy="${rpy}" />
         </joint>
     </xacro:macro>
-      <!-- common mecanum wheel link-->
+    <!-- common mecanum wheel link-->
     <xacro:macro name="common_mecanum_wheel_link" params="name material fdir *origin">
         <link name="${name}">
@@ -111,5 +118,5 @@
                 <pose>0 0 0 0 0 0</pose>
                 <geometry>
-                    <sphere radius="0.032391999999999997" />
+                    <sphere radius="0.04" />
                 </geometry>
             </collision>
@@ -121,14 +128,14 @@
                     <contact>
                         <ode />
-                      </contact>
-                  <friction>
-                    <ode>
-                      <mu>1.0</mu>
-                      <mu2>0.0</mu2>
-                      <fdir1 gz:expressed_in="base_footprint">${fdir}</fdir1>
-                    </ode>
-                  </friction>
+                    </contact>
+                    <friction>
+                        <ode>
+                            <mu>1.0</mu>
+                            <mu2>0.0</mu2>
+                            <fdir1 gz:expressed_in="base_footprint">${fdir}</fdir1>
+                        </ode>
+                    </friction>
                 </surface>
-              </collision>
+            </collision>
             <!-- <mu1>1</mu1>
             <mu2>0</mu2>
@@ -159,54 +166,88 @@
         </inertial>
     </common_link>
-    <fixed_joint name="base_joint" parent="base_footprint" child="base_link" xyz="0.0 0.0 0.076" rpy="0 0 0"/> -->
-    <!-- <fixed_joint name="base_imu" parent="base_link" child="imu_link" xyz="0.001 0.017 0.0322" rpy="0 3.1415 1.5707"/> -->
-    <xacro:common_link name="laser_link" material="White" path="sensor">
-        <inertial>
-            <origin xyz="-0.0176558922685589 0.000671805271544437 0.0219302095894866" rpy="0 0 0"/>
-            <mass value="0.0483909504209895"/>
-            <inertia ixx="1.58456966399128E-05" ixy="-4.23913983850005E-07" ixz="-2.09597897904374E-07"
-                     iyy="3.89262522903605E-05" iyz="3.24809725932687E-07" izz="4.86230801106223E-05"/>
-        </inertial>
-    </xacro:common_link>
-    <xacro:fixed_joint name="laser_joint" parent="base_link" child="laser_link" xyz="0.10478 0 0.0471" rpy="0 0 0"/>
+    <fixed_joint name="base_joint" parent="base_footprint" child="base_link" xyz="0.0 0.0 0.076" rpy="0
+    0 0"/> -->
+    <link name="imu_link"/>
+    <!-- <xacro:fixed_joint name="base_imu" parent="base_link" child="imu_link" xyz="0 0 0"
+        rpy="0 3.1415 1.5707"/>  -->
+    <xacro:fixed_joint name="base_imu" parent="base_link" child="imu_link" xyz="0.001 0.017 0.0322"
+        rpy="0 3.1415 1.5707"/>
+   <link name="laser_link"/>
+    <xacro:common_link name="sllidar_link" material="White" path="sensor">
+        <inertial>
+            <origin xyz="-0.0176558922685589 0.000671805271544437 0.0219302095894866" rpy="0 0 0" />
+            <!-- <origin xyz="-0.0176558922685589 0.000671805271544437 0.0219302095894866" rpy="0 0 0" /> -->
+            <mass value="0.0483909504209895" />
+            <inertia ixx="1.58456966399128E-05" ixy="-4.23913983850005E-07"
+                ixz="-2.09597897904374E-07"
+                iyy="3.89262522903605E-05" iyz="3.24809725932687E-07" izz="4.86230801106223E-05" />
+        </inertial>
+    </xacro:common_link>
+    <xacro:fixed_joint name="sllidar_joint" parent="base_link" child="sllidar_link"
+        xyz="0.10478 0 0" rpy="0 0 0" />
+        <xacro:fixed_joint name="laser_joint" parent="base_link" child="laser_link"
+        xyz="0.10478 0 0.035" rpy="0 0 3.14159" />
+        <!-- xyz="0.10478 0 0.0471" rpy="0 0 0" /> -->
     <xacro:common_link name="camera_link" material="White" path="sensor">
         <inertial>
-            <origin xyz="0 0 0" rpy="0 0 0"/>
-            <mass value="0"/>
-            <inertia ixx="0" ixy="0" ixz="0" iyy="0" iyz="0" izz="0"/>
-        </inertial>
-    </xacro:common_link>
-    <xacro:fixed_joint name="camera_joint" parent="base_link" child="camera_link" xyz="-0.043645 0 0.41955" rpy="0 0 0"/>
+            <origin xyz="0 0 0" rpy="0 0 0" />
+            <mass value="0" />
+            <inertia ixx="0" ixy="0" ixz="0" iyy="0" iyz="0" izz="0" />
+        </inertial>
+    </xacro:common_link>
     <xacro:common_link name="arm_link1" material="White" path="X3plus">
         <inertial>
-            <origin xyz="1.99179507982521E-05 -5.98354652829568E-05 0.0114289358828097" rpy="0 0 0"/>
-            <mass value="0.0279545499871709"/>
-            <inertia
-                    ixx="1.19144359314975E-05"
-                    ixy="-9.26068510046816E-09"
-                    ixz="3.16060516198683E-09"
-                    iyy="1.05642517915377E-05"
-                    iyz="2.69674403668579E-08"
-                    izz="1.49639510661413E-05"/>
-        </inertial>
-    </xacro:common_link>
-    <xacro:revolute_joint name="arm_joint1" parent="base_link" child="arm_link1" xyz="0.09825 0 0.102" rpy="0 0 0" axisZ="-1"
-                    lower="-${pi/2}" upper="${pi/2}"/>
-    <xacro:common_link name="arm_link2" material="Green" path="X3plus">
-        <inertial>
-            <origin xyz="0.024903 -0.0022632 -0.00066663" rpy="0 0 0"/>
-            <mass value="0.031605"/>
-            <inertia
-                    ixx="5.8495E-06"
-                    ixy="-8.8092E-07"
-                    ixz="1.5336E-07"
-                    iyy="2.667E-05"
-                    iyz="7.1365E-09"
-                    izz="2.4695E-05"/>
-        </inertial>
-    </xacro:common_link>
-    <xacro:revolute_joint name="arm_joint2" parent="arm_link1" child="arm_link2" xyz="0 0 0.0405"
-                    rpy="-${pi/2} 0 0" axisZ="-1" lower="-${pi/2}" upper="${pi/2}"/>
-    <xacro:common_link name="arm_link3" material="White" path="X3plus">
+            <origin xyz="1.99179507982521E-05 -5.98354652829568E-05 0.0114289358828097" rpy="0 0 0" />
+            <mass value="0.0279545499871709" />
+            <inertia
+                ixx="1.19144359314975E-05"
+                ixy="-9.26068510046816E-09"
+                ixz="3.16060516198683E-09"
+                iyy="1.05642517915377E-05"
+                iyz="2.69674403668579E-08"
+                izz="1.49639510661413E-05" />
+        </inertial>
+    </xacro:common_link>
+    <xacro:if value="${fixedPLZJoints}">
+        <xacro:fixed_joint name="arm_joint1" parent="base_link" child="arm_link1"
+        xyz="0.09825 0 0.102" rpy="0 0 0" />
+    </xacro:if>
+    <xacro:unless value="${fixedPLZJoints}">
+        <xacro:revolute_joint name="arm_joint1" parent="base_link" child="arm_link1"
+        xyz="0.09825 0 0.102" rpy="0 0 0" axisZ="-1"
+        lower="-${pi/2}" upper="${pi/2}" />
+    </xacro:unless>
+    <xacro:common_link name="arm_link2b" material="Green" path="X3plus">
+        <inertial>
+            <origin xyz="0.024903 -0.0022632 -0.00066663" rpy="0 0 0" />
+            <mass value="0.031605" />
+            <inertia
+                ixx="5.8495E-06"
+                ixy="-8.8092E-07"
+                ixz="1.5336E-07"
+                iyy="2.667E-05"
+                iyz="7.1365E-09"
+                izz="2.4695E-05" />
+        </inertial>
+    </xacro:common_link>
+    <xacro:if value="${fixedPLZJoints}">
+        <xacro:fixed_joint name="arm_joint2" parent="arm_link1" child="arm_link2b" xyz="0 0 0.0405"
+        rpy="-${pi/2} 0 0"   />
+    </xacro:if>
+    <xacro:unless value="${fixedPLZJoints}">
+        <xacro:revolute_joint name="arm_joint2" parent="arm_link1" child="arm_link2b" xyz="0 0 0.0405"
+        rpy="-${pi/2} 0 0" axisZ="-1" lower="-${pi/2}" upper="${pi/2}" />
+    </xacro:unless>
+    <xacro:fixed_joint name="camera_joint" parent="arm_link2b" child="camera_link" xyz="0 -0.07 0"
+        rpy="${pi/2} 0 0" />
+    <!-- <xacro:fixed_joint name="camera_joint" parent="base_link" child="camera_link"
+        xyz="0.057105 1.7948E-05 0.03755" rpy="0 0 0" /> -->
+   <joint name="camera_optical_joint" type="fixed">
+            <origin xyz="0 0 0" rpy="${-pi/2} 0 ${-pi/2}" />
+            <parent link="camera_link" />
+            <child link="camera_link_optical" />
+        </joint>
+        <link name="camera_link_optical"></link>
+    <!-- <xacro:common_link name="arm_link3" material="White" path="X3plus">
         <inertial>
             <origin xyz="0.024903 -0.0022634 -0.0013962" rpy="0 0 0"/>
@@ -221,5 +262,6 @@
         </inertial>
     </xacro:common_link>
-    <xacro:revolute_joint name="arm_joint3" parent="arm_link2" child="arm_link3" xyz="0 -0.0829 0" rpy="0 0 0"
+    <xacro:revolute_joint name="arm_joint3" parent="arm_link2" child="arm_link3" xyz="0 -0.0829 0"
+    rpy="0 0 0"
                     axisZ="-1" lower="-${pi/2}" upper="${pi/2}"/>
     <xacro:common_link name="arm_link4" material="Green" path="X3plus">
@@ -236,5 +278,6 @@
         </inertial>
     </xacro:common_link>
-    <xacro:revolute_joint name="arm_joint4" parent="arm_link3" child="arm_link4" xyz="0 -0.0829 0" rpy="0 0 0"
+    <xacro:revolute_joint name="arm_joint4" parent="arm_link3" child="arm_link4" xyz="0 -0.0829 0"
+    rpy="0 0 0"
                     axisZ="-1" lower="-${pi/2}" upper="${pi/2}"/>
     <xacro:common_link name="arm_link5" material="White" path="X3plus">
@@ -251,5 +294,6 @@
         </inertial>
     </xacro:common_link>
-    <xacro:revolute_joint name="arm_joint5" parent="arm_link4" child="arm_link5" xyz="-0.00215 -0.17455 0"
+    <xacro:revolute_joint name="arm_joint5" parent="arm_link4" child="arm_link5" xyz="-0.00215 -0.17455
+    0"
                     rpy="${pi/2} 0 0" axisZ="1" lower="-${pi/2}" upper="${pi}"/>
     <xacro:common_link name="rlink1" material="Green" path="X3plus">
@@ -266,5 +310,6 @@
         </inertial>
     </xacro:common_link>
-    <xacro:revolute_joint name="grip_joint" parent="arm_link5" child="rlink1" xyz="-0.0035 -0.012625 -0.0685"
+    <xacro:revolute_joint name="grip_joint" parent="arm_link5" child="rlink1" xyz="-0.0035 -0.012625
+    -0.0685"
                     rpy="0 -${pi/2} 0" axisZ="1" lower="-${pi/2}" upper="0"/>
     <xacro:common_link name="rlink2" material="Green" path="X3plus">
@@ -281,5 +326,6 @@
         </inertial>
     </xacro:common_link>
-    <xacro:continuous_joint name="rlink_joint2" parent="rlink1" child="rlink2" xyz="0.03 -0.00075429 0" rpy="0 0 0" mimic="-1"/>
+    <xacro:continuous_joint name="rlink_joint2" parent="rlink1" child="rlink2" xyz="0.03 -0.00075429 0"
+    rpy="0 0 0" mimic="-1"/>
     <xacro:common_link name="rlink3" material="Green" path="X3plus">
         <inertial>
@@ -295,5 +341,6 @@
         </inertial>
     </xacro:common_link>
-    <xacro:continuous_joint name="rlink_joint3" parent="arm_link5" child="rlink3" xyz="-0.0035 -0.0045 -0.0505"
+    <xacro:continuous_joint name="rlink_joint3" parent="arm_link5" child="rlink3" xyz="-0.0035 -0.0045
+    -0.0505"
                       rpy="0 -${pi/2} 0" mimic="1"/>
     <xacro:common_link name="llink1" material="Green" path="X3plus">
@@ -310,5 +357,6 @@
         </inertial>
     </xacro:common_link>
-    <xacro:continuous_joint name="llink_joint1" parent="arm_link5" child="llink1" xyz="-0.0035 0.012375 -0.0685"
+    <xacro:continuous_joint name="llink_joint1" parent="arm_link5" child="llink1" xyz="-0.0035 0.012375
+    -0.0685"
                       rpy="0 -${pi/2} 0" mimic="-1"/>
     <xacro:common_link name="llink2" material="Green" path="X3plus">
@@ -320,5 +368,6 @@
         </inertial>
     </xacro:common_link>
-    <xacro:continuous_joint name="llink_joint2" parent="llink1" child="llink2" xyz="0.03 0.00065104 0" rpy="0 0 0"
+    <xacro:continuous_joint name="llink_joint2" parent="llink1" child="llink2" xyz="0.03 0.00065104 0"
+    rpy="0 0 0"
                       mimic="1"/>
     <xacro:common_link name="llink3" material="Green" path="X3plus">
@@ -330,5 +379,6 @@
         </inertial>
     </xacro:common_link>
-    <xacro:continuous_joint name="llink_joint3" parent="arm_link5" child="llink3" xyz="-0.0035 0.0045 -0.0505"
+    <xacro:continuous_joint name="llink_joint3" parent="arm_link5" child="llink3" xyz="-0.0035 0.0045
+    -0.0505"
                       rpy="0 -${pi/2} 0" mimic="-1"/>
     <xacro:common_link name="mono_link" material="White" path="sensor">
@@ -340,43 +390,45 @@
         </inertial>
     </xacro:common_link>
-    <xacro:fixed_joint name="mono_joint" parent="arm_link4" child="mono_link" xyz="-0.0481 -0.05145 -0.0022"
+    <xacro:fixed_joint name="mono_joint" parent="arm_link4" child="mono_link" xyz="-0.0481 -0.05145
+    -0.0022"
                  rpy="${pi/2} 0 0"/>
-   <xacro:common_mecanum_wheel_link name="front_right_wheel" material="White" fdir="1 1 0">
-            <inertial>
-                <origin xyz="1.9051E-06 -2.3183E-07 -0.00064079" rpy="0 0 0" />
-                <mass value="0.051532" />
-                <inertia ixx="1.4595E-05" ixy="-4.3975E-10" ixz="4.415E-10"
-                    iyy="1.4594E-05" iyz="-1.7476E-09" izz="2.4264E-05" />
-            </inertial>
-        </xacro:common_mecanum_wheel_link>
-        <xacro:common_mecanum_wheel_link name="front_left_wheel" material="White" fdir="1 -1 0">
-            <inertial>
-                <origin xyz="2.3728E-06 -9.4228E-07 0.00064068" rpy="0 0 0" />
-                <mass value="0.051543" />
-                <inertia ixx="1.4597E-05" ixy="-4.7945E-10" ixz="-2.4786E-10"
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
Commit message: Adding a april calibration tag

File: x3plus_description/urdf/yahboomcar_X3plus.urdf.xacro (robot description, xacro)
@@ -4,7 +4,8 @@
     <!-- define the list of relevant args -->
     <xacro:arg name="fixedPLZJoints" default="true" />
-    <xacro:arg name="fixedPLZJoints" default="true"  />
+    <xacro:arg name="addCalibration" default="true" />
     <!-- set the internal properties based on the arguments -->
     <xacro:property name="fixedPLZJoints" value="$(arg fixedPLZJoints)" />
+    <xacro:property name="addCalibration" value="$(arg addCalibration)" />
     <!-- <xacro:if value="${namespace == 'None'}">
         <xacro:property name="ns" value="" />
@@ -442,4 +443,10 @@
         child="back_left_wheel"
         xyz="-0.115  0.103 -0.038" rpy="-${pi/2} 0 0" axis="0 0 1" />
+    <xacro:if value="${addCalibration}">
+        <xacro:include filename="$(find x3plus_description)/urdf/calibration/apriltag_marker.xacro" />
+        <xacro:apriltag_marker namespace="" name="calibration_tag" parent="base_link" family="36_11" ID="1" size="0.1">
+                    <origin xyz="0 0 0.2" rpy=" 0 0 0" />
+        </xacro:apriltag_marker>
+    </xacro:if>
    <gazebo>
             <plugin name='gz::sim::systems::MecanumDrive' filename='gz-sim-mecanum-drive-system'>
@@ -488,5 +495,5 @@
         <publish_model_pose>: Set to true to publish model pose.
         <publish_nested_model_pose>: Set to true to publish nested model pose. The pose of the model that contains this system is also published unless publish_model_pose is set to false
-        <use_pose_vector_msg>: Set to true to publish a gz::msgs::Pose_V message instead of mulitple gz::msgs::Pose messages.
+        <use_pose_vector_msg>: Set to true to publish a gz::msgs::Pose_V message instead of multiple gz::msgs::Pose messages.
         <update_frequency>: Frequency of pose publications in Hz. A negative frequency publishes as fast as possible (i.e, at the rate of the simulation step)
         <static_publisher>: Set to true to publish static poses on a "<scoped_entity_name>/pose_static" topic. This will cause only dynamic poses to be published on the "<scoped_entity_name>/pose" topic.
