Commit message: Update URDF for PTZ Unit

File: x3plus_description/urdf/yahboomcar_X3plus.urdf.xacro (robot description, xacro)
@@ -3,8 +3,8 @@
     xmlns:gz="http://gazebosim.org/schema">
     <!-- define the list of relevant args -->
-    <xacro:arg name="fixedPLZJoints" default="true" />
+    <!-- <xacro:arg name="fixedPLZJoints" default="true" /> -->
     <xacro:arg name="addCalibration" default="true" />
     <!-- set the internal properties based on the arguments -->
-    <xacro:property name="fixedPLZJoints" value="$(arg fixedPLZJoints)" />
+    <!-- <xacro:property name="fixedPLZJoints" value="$(arg fixedPLZJoints)" /> -->
     <xacro:property name="addCalibration" value="$(arg addCalibration)" />
     <!-- <xacro:if value="${namespace == 'None'}">
@@ -210,13 +210,13 @@
         </inertial>
     </xacro:common_link>
-    <xacro:if value="${fixedPLZJoints}">
+    <!-- <xacro:if value="${fixedPLZJoints}">
         <xacro:fixed_joint name="arm_joint1" parent="base_link" child="arm_link1"
         xyz="0.09825 0 0.102" rpy="0 0 0" />
     </xacro:if>
-    <xacro:unless value="${fixedPLZJoints}">
+    <xacro:unless value="${fixedPLZJoints}"> -->
         <xacro:revolute_joint name="arm_joint1" parent="base_link" child="arm_link1"
         xyz="0.09825 0 0.102" rpy="0 0 0" axisZ="-1"
         lower="-${pi/2}" upper="${pi/2}" />
-    </xacro:unless>
+    <!-- </xacro:unless> -->
     <xacro:common_link name="arm_link2b" material="Green" path="X3plus">
         <inertial>
@@ -232,12 +232,12 @@
         </inertial>
     </xacro:common_link>
-    <xacro:if value="${fixedPLZJoints}">
+    <!-- <xacro:if value="${fixedPLZJoints}">
         <xacro:fixed_joint name="arm_joint2" parent="arm_link1" child="arm_link2b" xyz="0 0 0.0405"
         rpy="-${pi/2} 0 0"   />
     </xacro:if>
-    <xacro:unless value="${fixedPLZJoints}">
+    <xacro:unless value="${fixedPLZJoints}"> -->
         <xacro:revolute_joint name="arm_joint2" parent="arm_link1" child="arm_link2b" xyz="0 0 0.0405"
         rpy="-${pi/2} 0 0" axisZ="-1" lower="-${pi/2}" upper="${pi/2}" />
-    </xacro:unless>
+    <!-- </xacro:unless> -->
     <xacro:fixed_joint name="camera_joint" parent="arm_link2b" child="camera_link" xyz="0 -0.07 0"
         rpy="${pi/2} 0 0" />
@@ -483,8 +483,18 @@
             <joint_name>: Name of a joint to publish. This parameter can be specified multiple times, and is optional. All joints in a model will be published if joint names are not specified.
          -->
-      <plugin
-        filename="gz-sim-joint-state-publisher-system"
-        name="gz::sim::systems::JointStatePublisher">
-      </plugin>
+        <plugin
+            filename="gz-sim-joint-state-publisher-system"
+            name="gz::sim::systems::JointStatePublisher">
+        </plugin>
+        <plugin
+            filename="gz-sim-joint-position-controller-system"
+            name="gz::sim::systems::JointPositionController">
+            <joint_name>arm_joint1</joint_name>
+        </plugin>
+        <plugin
+            filename="gz-sim-joint-position-controller-system"
+            name="gz::sim::systems::JointPositionController">
+            <joint_name>arm_joint2b</joint_name>
+        </plugin>
       <!--
         Pose publisher system. Attach to an entity to publish the transform of its child entities in the form of gz::msgs::Pose messages, or a single gz::msgs::Pose_V message if "use_pose_vector_msg" is true.

Commit message: Add localization support and update EKF configurations
- Introduced 'use_localization' launch argument in bringup and journey launch files.
- Updated EKF configuration files to improve sensor integration and added a new ground truth EKF config.
- Modified robot description to adjust wheel radius and mass for better simulation accuracy.
- Adjusted frontier exploration parameters for improved navigation performance.
- Created a new launch file for ground truth localization.

File: x3plus_description/urdf/yahboomcar_X3plus.urdf.xacro (robot description, xacro)
@@ -21,10 +21,12 @@
     </material>
     <xacro:property name="ns" value="$(arg ns)" />
-    <xacro:property name="wheel_radius" value="0.05" />
+    <xacro:property name="wheel_radius" value="0.04" />
+    <!-- The base_footprint link must be a purely virtual mathematical frame projected
+     flat on the ground plane. It should never have physical substance. -->
     <link name="base_footprint" />
     <link name="base_link">
         <inertial>
             <origin xyz="-0.0304416859098744 4.23384368655101E-05 0.0448234503408059" rpy="0 0 0" />
-            <mass value="1.0754239466482" />
+            <mass value="1.5" />
             <inertia
                 ixx="0.0208831789264125"
@@ -53,8 +55,17 @@
         </collision>
     </link>
+    <!-- The joint connecting base_footprint to base_link must always be a fixed joint. -->
     <joint name="base_joint" type="fixed">
         <parent link="base_footprint" />
         <child link="base_link" />
-        <origin xyz="0.0 0.0 0.076" rpy="0 0 0" />
+        <!--
+        If your wheel radius is 0.040 (40mm), your base_link origin must be elevated
+        on the Z-axis by exactly the height of your axle center relative to the ground.
+        If your offset is set too low (e.g., 0.0 or 0.02), Gazebo spawns the heavy
+        chassis inside the ground plane. The physics engine panics, tries to push it out,
+         and causes endless jumping.
+         -->
+        <origin xyz="0.0 0.0 0.08" rpy="0 0 0" />
+        <!-- <origin xyz="0.0 0.0 0.076" rpy="0 0 0" /> -->
     </joint>
     <!-- common link-->
@@ -128,5 +139,12 @@
                 <surface>
                     <contact>
-                        <ode />
+                        <ode>
+                            <!-- Contact spring-damper for wheel-ground interaction -->
+                             <!-- Add contact stiffness (kp) and damping (kd) to your wheel links.
+                              This gives the tires a bit of simulated rubber "squish" to absorb
+                              physics jitter: -->
+                            <kp>1.0e5</kp>
+                            <kd>10.0</kd>
+                        </ode>
                     </contact>
                     <friction>
@@ -499,23 +517,46 @@
     </xacro:if>
         <gazebo>
-            <plugin name='gz::sim::systems::MecanumDrive' filename='gz-sim-mecanum-drive-system'>
+            <plugin name='gz::sim::systems::DiffDrive' filename='gz-sim-diff-drive-system'>
+                <left_joint>front_left_joint</left_joint>
+                <left_joint>back_left_joint</left_joint>
+                <right_joint>front_right_joint</right_joint>
+                <right_joint>back_right_joint</right_joint>
+                <!-- Lateral distance between left and right wheels -->
+                 <!-- end 2 end is 245.6 mm ; width of the wheel is 37.4 ==> 0.2082 -->
+                <wheel_separation>0.2082</wheel_separation>
+                <!-- Wheel radius -->
+                <wheel_radius>0.040</wheel_radius>
+                <odom_publish_frequency>20</odom_publish_frequency>
+                <odom_topic>/wheel/odometry</odom_topic>
+                <!--
+                Using the Robot Localization Package (EKF), ensure your individual sensor plugins
+                (like Gazebo differential drive plugins or IMUs) have their publish_tf parameter
+                set to false.
+                Only the EKF node should publish the final odom -> base_footprint transform.
+                -->
+                <publish_odom_tf>false</publish_odom_tf>
+                <topic>/cmd_vel</topic>
+                <!-- <tf_topic>/pose</tf_topic> -->
+            </plugin>
+<!--
+ <plugin name='gz::sim::systems::MecanumDrive' filename='gz-sim-mecanum-drive-system'>
                 <front_left_joint>front_left_joint</front_left_joint>
                 <front_right_joint>front_right_joint</front_right_joint>
                 <back_left_joint>back_left_joint</back_left_joint>
                 <back_right_joint>back_right_joint</back_right_joint>
-                <!-- Lateral distance between left and right wheels -->
-                 <!-- end 2 end is 245.6 mm ; width of the wheel is 37.4 ==> 0.2082 -->
+                <!- - Lateral distance between left and right wheels - ->
+                 <!- - end 2 end is 245.6 mm ; width of the wheel is 37.4 ==> 0.2082 - ->
                 <wheel_separation>0.2082</wheel_separation>
-                <!-- Longitudinal distance between front and back wheels -->
+                <!- - Longitudinal distance between front and back wheels - ->
                 <wheelbase>0.22</wheelbase>
-                <!-- Wheel radius -->
+                <!- - Wheel radius - ->
                 <wheel_radius>0.040</wheel_radius>
                 <min_acceleration>-5</min_acceleration>
                 <max_acceleration>5</max_acceleration>
-                <!-- <max_velocity>3.0</max_velocity>
-                <min_velocity>-3.0</min_velocity> -->
-                <!-- <min_jerk>3</min_jerk>
-                <max_jerk>-3</max_jerk> -->
-                <odom_publish_frequency>10</odom_publish_frequency>
+                <!- - <max_velocity>3.0</max_velocity>
+                <min_velocity>-3.0</min_velocity> - ->
+                <!- - <min_jerk>3</min_jerk>
+                <max_jerk>-3</max_jerk> - ->
+                <odom_publish_frequency>20</odom_publish_frequency>
                 <odom_topic>/wheel/odometry</odom_topic>
                 <publish_odom_tf>false</publish_odom_tf>
@@ -523,5 +564,5 @@
                 <topic>/cmd_vel</topic>
                 <tf_topic>/pose</tf_topic>
-            </plugin>
+            </plugin> -->
         <!--
             The JointStatePublisher system publishes joint state information for a model. The published message type is gz::msgs::Model, and the publication topic is determined by the <topic> parameter.
@@ -700,5 +741,5 @@
         <sensor name="imu_sensor" type="imu">
             <always_on>1</always_on>
-            <update_rate>10</update_rate>
+            <update_rate>20</update_rate>
             <visualize>true</visualize>
             <topic>imu</topic>
