Commit message: Fine tune SDF settings

File: x3plus_description/urdf/calibration/apriltag_marker.xacro (robot description, xacro)
@@ -57,5 +57,5 @@
         <mass value="0.001" />
         <origin xyz="0 0 0" rpy="0 0 0" />
-        <inertia ixx="0.00001" ixy="0" ixz="0" iyy="0.00001" iyz="0" izz="0.00002" />
+        <inertia ixx="0.00001" ixy="0.00001" ixz="0.00001" iyy="0.00001" iyz="0" izz="0.00002" />
       </inertial>
       <collision>

File: x3plus_description/urdf/yahboomcar_X3plus.urdf.xacro (robot description, xacro)
@@ -169,10 +169,58 @@
     <fixed_joint name="base_joint" parent="base_footprint" child="base_link" xyz="0.0 0.0 0.076" rpy="0
     0 0"/> -->
-    <link name="imu_link"/>
+    <!--
+    what counts as a valid inertia block for a “logical link” in SDF when the link has no physical geometry.
+    Harmonic enforces:
+        SDF 1.10 schema
+        Non‑zero mass for dynamic links
+        Positive‑definite inertia
+        No missing inertial blocks
+        No implicit defaults
+    -->
+    <link name="imu_link">
+        <inertial>
+            <mass value="0.0001"/>
+            <inertia
+                ixx="1e-6"
+                iyy="1e-6"
+                izz="1e-6"
+                ixy="0"
+                ixz="0"
+                iyz="0"/>
+        </inertial>
+    </link>
     <!-- <xacro:fixed_joint name="base_imu" parent="base_link" child="imu_link" xyz="0 0 0"
         rpy="0 3.1415 1.5707"/>  -->
     <xacro:fixed_joint name="base_imu" parent="base_link" child="imu_link" xyz="0.001 0.017 0.0322"
         rpy="0 3.1415 1.5707"/>
-   <link name="laser_link"/>
+   <link name="laser_link">
+           <inertial>
+            <mass value="0.0001"/>
+            <inertia
+                ixx="1e-6"
+                iyy="1e-6"
+                izz="1e-6"
+                ixy="0"
+                ixz="0"
+                iyz="0"/>
+        </inertial>
+        <!--
+        we use a very small sphere for the laser link, so that Gazebo can put the laser sensor on it.
+        The actual geometry of the laser is defined in the Gazebo sensor plugin.
+        Harmonic’s sensor system attaches sensors to renderable entities.
+        A link with no geometry is considered “non-renderable” and is skipped.
+        Adding a tiny sphere makes the link renderable, so the sensor is created.
+        -->
+        <visual>
+            <geometry>
+            <sphere radius="0.0001"/>
+            </geometry>
+        </visual>
+        <collision>
+            <geometry>
+            <sphere radius="0.0001"/>
+            </geometry>
+        </collision>
+    </link>
     <xacro:common_link name="sllidar_link" material="White" path="sensor">
         <inertial>
@@ -187,5 +235,5 @@
     <xacro:fixed_joint name="sllidar_joint" parent="base_link" child="sllidar_link"
         xyz="0.10478 0 0" rpy="0 0 0" />
-        <xacro:fixed_joint name="laser_joint" parent="base_link" child="laser_link"
+    <xacro:fixed_joint name="laser_joint" parent="base_link" child="laser_link"
         xyz="0.10478 0 0.035" rpy="0 0 3.14159" />
         <!-- xyz="0.10478 0 0.0471" rpy="0 0 0" /> -->
@@ -193,6 +241,6 @@
         <inertial>
             <origin xyz="0 0 0" rpy="0 0 0" />
-            <mass value="0" />
-            <inertia ixx="0" ixy="0" ixz="0" iyy="0" iyz="0" izz="0" />
+            <mass value="0.0001" />
+            <inertia ixx="1e-6" ixy="1e-6" ixz="1e-6" iyy="0" iyz="0" izz="0" />
         </inertial>
     </xacro:common_link>
@@ -450,5 +498,5 @@
         </xacro:apriltag_marker>
     </xacro:if>
-   <gazebo>
+        <gazebo>
             <plugin name='gz::sim::systems::MecanumDrive' filename='gz-sim-mecanum-drive-system'>
                 <front_left_joint>front_left_joint</front_left_joint>
@@ -476,6 +524,4 @@
                 <tf_topic>/pose</tf_topic>
             </plugin>
-        </gazebo>
-    <gazebo>
         <!--
             The JointStatePublisher system publishes joint state information for a model. The published message type is gz::msgs::Model, and the publication topic is determined by the <topic> parameter.
@@ -569,4 +615,76 @@
       </plugin> -->
     </gazebo>
+     <!-- <sensor name="magnetometer" type="magnetometer">
+          <always_on>1</always_on>
+          <update_rate>100</update_rate>
+          <visualize>true</visualize>
+          <topic>magnetometer</topic>
+          <enable_metrics>true</enable_metrics>
+          <magnetometer>
+            <x>
+              <noise type="gaussian">
+                <mean>0.0</mean>
+                <stddev>0.1</stddev>
+              </noise>
+            </x>
+            <y>
+              <noise type="gaussian">
+                <mean>0.0</mean>
+                <stddev>0.1</stddev>
+              </noise>
+            </y>
+            <z>
+              <noise type="gaussian">
+                <mean>0.0</mean>
+                <stddev>0.1</stddev>
+              </noise>
+            </z>
+          </magnetometer>
+        </sensor> -->
+    <gazebo reference="laser_link">
+        <sensor name='gpu_lidar' type='gpu_lidar'>
+            <pose>0 0 0 0 0 0</pose>
+            <!-- <pose relative_to='laser_link'>0 0 0 0 0 0</pose> -->
+            <topic>lidar</topic>
+            <update_rate>10</update_rate>
+            <!--
+                When using the following frame_id, the following error is shown during the launch in rviz2:
+                [rviz2-5] [INFO] [1745951906.206204296] [rviz]: Message Filter dropping message: frame 'x3plus_bot/base_footprint/gpu_lidar'
+                at time 73.900 for reason 'the timestamp on the message is earlier than all the data in the transform cache'
+                Which is caused by the fact that the frame_id is not set to the correct frame id
+                So when using the gz_frame_id, the following warning is shown:
+                [ruby $(which gz) sim-1] Warning [Utils.cc:132] [/sdf/model[@name="yahboomcar_X3plus"]/link[@name="base_footprint"]/sensor[@name="gpu_lidar"]/gz_frame_id:<urdf-string>:L0]: XML Element[gz_frame_id], child of element[sensor], not defined in SDF. Copying[gz_frame_id] as children of [sensor].
+            -->
+            <!-- <frame_id >laser_link</frame_id > -->
+            <gz_frame_id>laser_link</gz_frame_id >
+                <ray>
+                    <scan>
+                        <horizontal>
+                            <samples>720</samples>
+                            <resolution>1</resolution>
+                            <min_angle>-3.14159</min_angle>
+                            <max_angle>3.14159</max_angle>
+                            <!--
+                            <min_angle>-1.396263</min_angle>
+                            <max_angle>1.396263</max_angle>
+                            -->
+                        </horizontal>
+                        <!-- <vertical>
+                            <samples>1</samples>
+                            <resolution>0.01</resolution>
+                            <min_angle>0</min_angle>
+                            <max_angle>0</max_angle>
+                        </vertical> -->
+                    </scan>
+                    <range>
+                        <min>0.05</min>
+                        <max>16.0</max>
+                        <resolution>0.01</resolution>
+                    </range>
+                </ray>
+            <always_on>1</always_on>
+            <visualize>true</visualize>
+        </sensor>
+    </gazebo>
     <gazebo reference="imu_link">
         <sensor name="imu_sensor" type="imu">
@@ -633,76 +751,4 @@
                 </linear_acceleration>
               </imu>
-        </sensor>
-    </gazebo>
-     <!-- <sensor name="magnetometer" type="magnetometer">
-          <always_on>1</always_on>
-          <update_rate>100</update_rate>
-          <visualize>true</visualize>
-          <topic>magnetometer</topic>
-          <enable_metrics>true</enable_metrics>
-          <magnetometer>
-            <x>
-              <noise type="gaussian">
-                <mean>0.0</mean>
-                <stddev>0.1</stddev>
-              </noise>
-            </x>
-            <y>
-              <noise type="gaussian">
-                <mean>0.0</mean>
-                <stddev>0.1</stddev>
-              </noise>
-            </y>
-            <z>
-              <noise type="gaussian">
-                <mean>0.0</mean>
-                <stddev>0.1</stddev>
-              </noise>
-            </z>
-          </magnetometer>
-        </sensor> -->
-    <gazebo reference="laser_link">
-        <sensor name='gpu_lidar' type='gpu_lidar'>
-            <pose relative_to='laser_link'>0 0 0 0 0 0</pose>
-            <!-- <pose relative_to='laser_link'>0 0 0 0 0 0</pose> -->
-            <topic>lidar</topic>
-            <update_rate>10</update_rate>
-            <!--
-                When using the following frame_id, the following error is shown during the launch in rviz2:
-                [rviz2-5] [INFO] [1745951906.206204296] [rviz]: Message Filter dropping message: frame 'x3plus_bot/base_footprint/gpu_lidar'
-                at time 73.900 for reason 'the timestamp on the message is earlier than all the data in the transform cache'
-                Which is caused by the fact that the frame_id is not set to the correct frame id
-                So when using the gz_frame_id, the following warning is shown:
-                [ruby $(which gz) sim-1] Warning [Utils.cc:132] [/sdf/model[@name="yahboomcar_X3plus"]/link[@name="base_footprint"]/sensor[@name="gpu_lidar"]/gz_frame_id:<urdf-string>:L0]: XML Element[gz_frame_id], child of element[sensor], not defined in SDF. Copying[gz_frame_id] as children of [sensor].
-            -->
-            <!-- <frame_id >laser_link</frame_id > -->
-            <gz_frame_id>laser_link</gz_frame_id >
-                <ray>
-                    <scan>
-                        <horizontal>
-                            <samples>720</samples>
-                            <resolution>1</resolution>
-                            <min_angle>-3.14159</min_angle>
-                            <max_angle>3.14159</max_angle>
-                            <!--
-                            <min_angle>-1.396263</min_angle>
-                            <max_angle>1.396263</max_angle>
-                            -->
-                        </horizontal>
-                        <vertical>
-                            <samples>1</samples>
-                            <resolution>0.01</resolution>
-                            <min_angle>0</min_angle>
-                            <max_angle>0</max_angle>
-                        </vertical>
-                    </scan>
-                    <range>
-                        <min>0.05</min>
-                        <max>16.0</max>
-                        <resolution>0.01</resolution>
-                    </range>
-                </ray>
-            <always_on>1</always_on>
-            <visualize>true</visualize>
         </sensor>
     </gazebo>
